File: Level_shifter.kicad_sch (KiCad schematic)
At the start: 6 parts, among them Q1 Q_NMOS_GSD

Commit message: Update of data for PCBA
Parts:
- renumbered Q1 to Q2, Q1 to Q3, R10 to R14, R10 to R15, R10 to R16, R10 to R17
Changed lines of the file:
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@@
   (symbol (lib_id "Device:Q_NMOS_GSD") (at 147.32 81.28 270) (unit 1)
     (in_bom yes) (on_board yes) (dnp no) (fields_autoplaced)
-    (property "Reference" "Q1" (at 147.32 87.63 90)
+    (property "Reference" "Q2" (at 147.32 87.63 90)
       (effects (font (size 1.27 1.27)))
     )
@@
     (instances
       (project "raspi_comm_if_hat"
-        (path "/756acdc9-6e12-4c33-b236-b5e247e5c2ec"
-          (reference "Q1") (unit 1)
-        )
         (path "/756acdc9-6e12-4c33-b236-b5e247e5c2ec/21f89c75-f7a5-4452-ab90-eaeb5895f083"
           (reference "Q2") (unit 1)
@@
   (symbol (lib_id "Device:R") (at 125.73 77.47 0) (unit 1)
     (in_bom yes) (on_board yes) (dnp no)
-    (property "Reference" "R10" (at 127.508 76.3016 0)
+    (property "Reference" "R14" (at 127.508 76.3016 0)
       (effects (font (size 1.27 1.27)) (justify left))
     )
@@
     (instances
       (project "raspi_comm_if_hat"
-        (path "/756acdc9-6e12-4c33-b236-b5e247e5c2ec"
-          (reference "R10") (unit 1)
-        )
         (path "/756acdc9-6e12-4c33-b236-b5e247e5c2ec/21f89c75-f7a5-4452-ab90-eaeb5895f083"
           (reference "R14") (unit 1)
@@
   (symbol (lib_id "Device:R") (at 156.21 77.47 0) (unit 1)
     (in_bom yes) (on_board yes) (dnp no)
-    (property "Reference" "R10" (at 157.988 76.3016 0)
+    (property "Reference" "R16" (at 157.988 76.3016 0)
       (effects (font (size 1.27 1.27)) (justify left))
     )
@@
     (instances
       (project "raspi_comm_if_hat"
-        (path "/756acdc9-6e12-4c33-b236-b5e247e5c2ec"
-          (reference "R10") (unit 1)
-        )
         (path "/756acdc9-6e12-4c33-b236-b5e247e5c2ec/21f89c75-f7a5-4452-ab90-eaeb5895f083"
           (reference "R16") (unit 1)
@@
   (symbol (lib_id "Device:Q_NMOS_GSD") (at 133.35 92.71 270) (unit 1)
     (in_bom yes) (on_board yes) (dnp no) (fields_autoplaced)
-    (property "Reference" "Q1" (at 133.35 99.06 90)
+    (property "Reference" "Q3" (at 133.35 99.06 90)
       (effects (font (size 1.27 1.27)))
     )
@@
     (instances
       (project "raspi_comm_if_hat"
-        (path "/756acdc9-6e12-4c33-b236-b5e247e5c2ec"
-          (reference "Q1") (unit 1)
-        )
         (path "/756acdc9-6e12-4c33-b236-b5e247e5c2ec/21f89c75-f7a5-4452-ab90-eaeb5895f083"
           (reference "Q3") (unit 1)
@@
   (symbol (lib_id "Device:R") (at 165.1 77.47 0) (unit 1)
     (in_bom yes) (on_board yes) (dnp no)
-    (property "Reference" "R10" (at 166.878 76.3016 0)
+    (property "Reference" "R17" (at 166.878 76.3016 0)
       (effects (font (size 1.27 1.27)) (justify left))
     )
@@
     (instances
       (project "raspi_comm_if_hat"
-        (path "/756acdc9-6e12-4c33-b236-b5e247e5c2ec"
-          (reference "R10") (unit 1)
-        )
         (path "/756acdc9-6e12-4c33-b236-b5e247e5c2ec/21f89c75-f7a5-4452-ab90-eaeb5895f083"
           (reference "R17") (unit 1)
@@
   (symbol (lib_id "Device:R") (at 138.43 77.47 0) (unit 1)
     (in_bom yes) (on_board yes) (dnp no)
-    (property "Reference" "R10" (at 140.208 76.3016 0)
+    (property "Reference" "R15" (at 140.208 76.3016 0)
       (effects (font (size 1.27 1.27)) (justify left))
     )
@@
     (instances
       (project "raspi_comm_if_hat"
-        (path "/756acdc9-6e12-4c33-b236-b5e247e5c2ec"
-          (reference "R10") (unit 1)
-        )
         (path "/756acdc9-6e12-4c33-b236-b5e247e5c2ec/21f89c75-f7a5-4452-ab90-eaeb5895f083"
           (reference "R15") (unit 1)

Commit message: Add LSCS
Parts:
- Q2, Q3: LCSC (none) -> C7420339
- R14, R15, R16, R17: footprint Resistor_SMD:R_0603_1608Metric_Pad0.98x0.95mm_HandSolder -> Resistor_SMD:R_0402_1005Metric; LCSC (none) -> C25744
Changed lines of the file:
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@@
+      (effects (font (size 1.27 1.27)) hide)
+    )
+    (property "LCSC" "C7420339" (at 147.32 81.28 0)
       (effects (font (size 1.27 1.27)) hide)
     )
@@
       (effects (font (size 1.27 1.27)) (justify left))
     )
-    (property "Footprint" "Resistor_SMD:R_0603_1608Metric_Pad0.98x0.95mm_HandSolder" (at 123.952 77.47 90)
+    (property "Footprint" "Resistor_SMD:R_0402_1005Metric" (at 123.952 77.47 90)
       (effects (font (size 1.27 1.27)) hide)
     )
     (property "Datasheet" "~" (at 125.73 77.47 0)
+      (effects (font (size 1.27 1.27)) hide)
+    )
+    (property "LCSC" "C25744" (at 125.73 77.47 0)
       (effects (font (size 1.27 1.27)) hide)
     )
@@
       (effects (font (size 1.27 1.27)) (justify left))
     )
-    (property "Footprint" "Resistor_SMD:R_0603_1608Metric_Pad0.98x0.95mm_HandSolder" (at 154.432 77.47 90)
+    (property "Footprint" "Resistor_SMD:R_0402_1005Metric" (at 154.432 77.47 90)
       (effects (font (size 1.27 1.27)) hide)
     )
     (property "Datasheet" "~" (at 156.21 77.47 0)
+      (effects (font (size 1.27 1.27)) hide)
+    )
+    (property "LCSC" "C25744" (at 156.21 77.47 0)
       (effects (font (size 1.27 1.27)) hide)
     )
@@
       (effects (font (size 1.27 1.27)) hide)
     )
+    (property "LCSC" "C7420339" (at 133.35 92.71 0)
+      (effects (font (size 1.27 1.27)) hide)
+    )
     (pin "1")
     (pin "3")
@@
       (effects (font (size 1.27 1.27)) (justify left))
     )
-    (property "Footprint" "Resistor_SMD:R_0603_1608Metric_Pad0.98x0.95mm_HandSolder" (at 163.322 77.47 90)
+    (property "Footprint" "Resistor_SMD:R_0402_1005Metric" (at 163.322 77.47 90)
       (effects (font (size 1.27 1.27)) hide)
     )
     (property "Datasheet" "~" (at 165.1 77.47 0)
+      (effects (font (size 1.27 1.27)) hide)
+    )
+    (property "LCSC" "C25744" (at 165.1 77.47 0)
       (effects (font (size 1.27 1.27)) hide)
     )
@@
       (effects (font (size 1.27 1.27)) (justify left))
     )
-    (property "Footprint" "Resistor_SMD:R_0603_1608Metric_Pad0.98x0.95mm_HandSolder" (at 136.652 77.47 90)
+    (property "Footprint" "Resistor_SMD:R_0402_1005Metric" (at 136.652 77.47 90)
       (effects (font (size 1.27 1.27)) hide)
     )
@@
       (effects (font (size 1.27 1.27)) hide)
     )
+    (property "LCSC" "C25744" (at 138.43 77.47 0)
+      (effects (font (size 1.27 1.27)) hide)
+    )
